File: circuits/schematics/learning-kicad/learning-kicad.kicad_sch (KiCad schematic)
At the start: 12 parts, among them SW1 SW_Push, SW2 SW_Push, SW3 SW_Push

Commit message: Started learning PCB design
Parts:
- added SSD1: ~, sp02 stuff:SSD1306, symbol sp02 stuff:SSD1306
- added U1: ~, sp02 stuff:MAX30102, symbol sp02 stuff:MAX30102_Module
- C1, C2, C3: footprint (none) -> Capacitor_THT:C_Disc_D4.7mm_W2.5mm_P5.00mm
- D1: footprint (none) -> LED_THT:LED_D5.0mm
- R1, R2, R3, R4: footprint (none) -> Resistor_THT:R_Axial_DIN0207_L6.3mm_D2.5mm_P7.62mm_Horizontal
- SW1, SW2, SW3: footprint (none) -> Button_Switch_THT:SW_PUSH_6mm
Connections:
- net +5V: now also SSD1.2 (VCC), U1.5 (VCC)
- net GND: now also SSD1.1 (GND), U1.4 (GND)
- net at A1.13 (SDA/A4): now also SSD1.4 (SDA), U1.2 (SDA)
- net at A1.14 (SCL/A5): now also SSD1.3 (SCL), U1.3 (SCL)
- no-connect marks 0 -> 21
